Commit message: work for gazebo

File: spot_description/urdf/spot.urdf.xacro (robot description, xacro)
@@ -1,4 +1,5 @@
 <?xml version="1.0"?>
 <robot xmlns:xacro="http://www.ros.org/wiki/xacro" name="spot_quadruped">
+    <xacro:include filename="material.xacro"/>
     <xacro:property name="body_length" value="0.22"/>
     <xacro:property name="body_width" value="0.12"/>
@@ -14,19 +15,4 @@
     <xacro:property name="fuss_height" value="0.03"/>
     <xacro:property name="fuss_ballen" value="0.015"/>
-    <material name="black">
-        <color rgba=" 0 0 0 1"/>
-    </material>
-    <material name="green">
-        <color rgba=" 0 1 0 1"/>
-    </material>
-    <material name="blue">
-        <color rgba=" 0 0 1 1"/>
-    </material>
-    <material name="red">
-        <color rgba=" 1 0 0 1"/>
-    </material>
-    <material name="white">
-        <color rgba=" 1 1 1 1"/>
-    </material>
     <link name="base_footprint"/>
     <link name="base_link">
@@ -39,4 +25,13 @@
             <material name="black"/>
         </visual>
+        <collision>
+            <origin xyz="0.0 0.0 ${body_width/2}" rpy="0.0 ${pi/2} 0.0 "/>
+            <geometry>
+                <cylinder radius="${body_height/2}" length="${body_length}"/>
+                <!--<box size="${body_length} ${body_width} ${body_height}"/> -->
+            </geometry>
+        </collision>
+        <xacro:cylinder_inertia m="0.5" r="${body_height/2}" h="${body_length}"
+                           xyz="0 0 0" rpy="0 0 0"/>
     </link>
     <joint name="virtuel_joint" type="fixed">
@@ -54,4 +49,12 @@
             </geometry>
         </visual>
+        <collision>
+            <origin xyz="0.0 0.0 0.0" rpy="0.0 0.0 0.0"/>
+            <geometry>
+                <box size="${shoulder_length} ${shoulder_width} ${shoulder_height}"/>
+            </geometry>
+        </collision>
+        <xacro:box_inertia m="0.1" l="${shoulder_length}" w="${shoulder_width}" h="${shoulder_height}"
+                           xyz="0 0 0" rpy="0 0 0"/>
     </link>
     </xacro:macro>
@@ -70,4 +73,12 @@
             <material name="white"/>
         </visual>
+        <collision>
+            <origin xyz="-0.03 0.0 0.0" rpy="0.0 0.0 0.0"/>
+            <geometry>
+                <box size="${bein_length}  ${bein_width} ${bein_height}"/>
+            </geometry>
+        </collision>
+        <xacro:box_inertia m="0.1" l="${bein_length}" w="${bein_width}" h="${bein_height}"
+                           xyz="0 0 0" rpy="0 0 0"/>
     </link>
     </xacro:macro>
@@ -86,4 +97,12 @@
             <material name="black"/>
         </visual>
+        <collision>
+            <origin xyz="0.055 0.0 0.0" rpy="0.0 0.0 0.0"/>
+            <geometry>
+                <box size="${fuss_length}  ${fuss_width} ${fuss_height}"/>
+            </geometry>
+        </collision>
+        <xacro:box_inertia m="0.1" l="${fuss_length}" w="${fuss_width}" h="${fuss_height}"
+                           xyz="0 0 0" rpy="0 0 0"/>
     </link>
     </xacro:macro>
@@ -102,4 +121,12 @@
             <material name="black"/>
         </visual>
+        <collision>
+            <origin xyz="-0.015 0.0 0.0" rpy="${pi/2} 0.0 0.0"/>
+            <geometry>
+                <cylinder radius="${fuss_ballen}" length="${fuss_width}"/>
+            </geometry>
+        </collision>
+        <xacro:cylinder_inertia m="0.01" r="${fuss_ballen}" h="${fuss_width}"
+                           xyz="0 0 0" rpy="0 0 0"/>
     </link>
     </xacro:macro>

Commit message: play with urdf

File: spot_description/urdf/spot.urdf.xacro (robot description, xacro)
@@ -15,11 +15,13 @@
     <xacro:property name="fuss_height" value="0.03"/>
     <xacro:property name="fuss_ballen" value="0.015"/>
+    <xacro:property name="scale" value="0.001 0.001 0.001"/>
     <link name="base_footprint"/>
     <link name="base_link">
         <visual>
-            <origin xyz="0.0 0.0 ${body_width/2}" rpy="0.0 ${pi/2} 0.0 "/>
-            <geometry>
-                <cylinder radius="${body_height/2}" length="${body_length}"/>
-                <!--<box size="${body_length} ${body_width} ${body_height}"/> -->
+            <origin xyz="-0.013 -0.0325 0.125" rpy="0.0 0.0 ${-pi/2} "/>
+            <geometry>
+               <cylinder radius="${body_height/2}" length="${body_length}"/>
+               <!-- <mesh filename="package://spot_description/meshes/Spot_Chassis.stl" scale="${scale}"/>
+                <box size="${body_length} ${body_width} ${body_height}"/> -->
             </geometry>
             <material name="black"/>
@@ -148,5 +150,5 @@
         <axis xyz="0 -1 0"/>
         <limit lower="0" upper="${pi/2}" velocity="50.0" effort="1000.0"/>
-        <origin xyz="0.0 -${shoulder_width/2 + bein_width/2 + 0.003} -0.01" rpy="0 0 0"/>
+        <origin xyz="0.0 -${shoulder_width/2 + bein_width/2 + 0.003} -0.01" rpy="0 ${-pi/2} 0"/>
     </joint>
     <joint name="joint_2" type="revolute">
@@ -155,5 +157,5 @@
         <axis xyz="0 1 0"/>
         <limit lower="0" upper="${pi/2}" velocity="50.0" effort="1000.0"/>
-        <origin xyz="-0.107 0.0 -0.03" rpy="0 0 0"/>
+        <origin xyz="-0.107 0.0 0.03" rpy="0 ${-pi/2} 0"/>
     </joint>
     <joint name="rechter_fuss_F_endpoint" type="fixed">
@@ -174,6 +176,6 @@
         <child link="front_l_bein_link"/>
         <axis xyz="0 -1 0"/>
-        <limit lower="0" upper="${pi/2}" velocity="50.0" effort="1000.0"/>
-        <origin xyz="0.0 ${shoulder_width/2 + bein_width/2 + 0.003} -0.01" rpy="0 0 0"/>
+        <limit lower="${-pi/4}" upper="${pi/4}" velocity="50.0" effort="1000.0"/>
+        <origin xyz="0.0 ${shoulder_width/2 + bein_width/2 + 0.003} -0.01" rpy="0 ${-pi/2} 0"/>
     </joint>
     <joint name="joint_5" type="revolute">
@@ -181,6 +183,6 @@
         <child link="front_l_fuss_link"/>
         <axis xyz="0 1 0"/>
-        <limit lower="0" upper="${pi/2}" velocity="50.0" effort="1000.0"/>
-        <origin xyz="-0.107 0.0 -0.03" rpy="0 0 0"/>
+        <limit lower="${-pi/4}" upper="${pi/4}" velocity="50.0" effort="1000.0"/>
+        <origin xyz="-0.107 0.0 0.03" rpy="0 ${-pi/2} 0"/>
     </joint>
     <joint name="linker_fuss_F_endpoint" type="fixed">
@@ -195,5 +197,5 @@
         <axis xyz="-1 0 0"/>
         <limit lower="${-pi/4}" upper="${pi/4}" velocity="50.0" effort="1000.0"/>
-        <origin xyz="-0.132 -0.0435 ${body_width/2}" rpy="0 0 0"/>
+        <origin xyz="-0.134 -0.0435 ${body_width/2}" rpy="0 0 0"/>
     </joint>
     <joint name="joint_7" type="revolute">
@@ -201,6 +203,6 @@
         <child link="heck_r_bein_link"/>
         <axis xyz="0 -1 0"/>
-        <limit lower="0" upper="${pi/2}" velocity="50.0" effort="1000.0"/>
-        <origin xyz="0.0 -${shoulder_width/2 + bein_width/2 + 0.003} -0.01" rpy="0 0 0"/>
+        <limit lower="${-pi/4}" upper="${pi/4}" velocity="50.0" effort="1000.0"/>
+        <origin xyz="0.0 -${shoulder_width/2 + bein_width/2 + 0.003} -0.01" rpy="0 ${-pi/2} 0"/>
     </joint>
     <joint name="joint_8" type="revolute">
@@ -208,6 +210,6 @@
         <child link="heck_r_fuss_link"/>
         <axis xyz="0 1 0"/>
-        <limit lower="0" upper="${pi/2}" velocity="50.0" effort="1000.0"/>
-        <origin xyz="-0.107 0.0 -0.03" rpy="0 0 0"/>
+        <limit lower="${-pi/4}" upper="${pi/4}" velocity="50.0" effort="1000.0"/>
+        <origin xyz="-0.107 0.0 0.03" rpy="0 ${-pi/2} 0"/>
     </joint>
     <joint name="rechter_fuss_H_endpoint" type="fixed">
@@ -222,5 +224,5 @@
         <axis xyz="1 0 0"/>
         <limit lower="${-pi/4}" upper="${pi/4}" velocity="50.0" effort="1000.0"/>
-        <origin xyz="-0.132 0.0435 ${body_width/2}" rpy="0 0 0"/>
+        <origin xyz="-0.134 0.0435 ${body_width/2}" rpy="0 0 0"/>
     </joint>
     <joint name="joint_10" type="revolute">
@@ -228,6 +230,6 @@
         <child link="heck_l_bein_link"/>
         <axis xyz="0 -1 0"/>
-        <limit lower="0" upper="${pi/2}" velocity="50.0" effort="1000.0"/>
-        <origin xyz="0.0 ${shoulder_width/2 + bein_width/2 + 0.003} -0.01" rpy="0 0 0"/>
+        <limit lower="${-pi/4}" upper="${pi/4}" velocity="50.0" effort="1000.0"/>
+        <origin xyz="0.0 ${shoulder_width/2 + bein_width/2 + 0.003} -0.01" rpy="0 ${-pi/2} 0"/>
     </joint>
     <joint name="joint_11" type="revolute">
@@ -235,6 +237,6 @@
         <child link="heck_l_fuss_link"/>
         <axis xyz="0 1 0"/>
-        <limit lower="0" upper="${pi/2}" velocity="50.0" effort="1000.0"/>
-        <origin xyz="-0.107 0.0 -0.03" rpy="0 0 0"/>
+        <limit lower="${-pi/4}" upper="${pi/4}" velocity="50.0" effort="1000.0"/>
+        <origin xyz="-0.107 0.0 0.03" rpy="0 ${-pi/2} 0"/>
     </joint>
     <joint name="linker_fuss_H_endpoint" type="fixed">

Commit message: in work

File: spot_description/urdf/spot.urdf.xacro (robot description, xacro)
@@ -2,246 +2,6 @@
 <robot xmlns:xacro="http://www.ros.org/wiki/xacro" name="spot_quadruped">
     <xacro:include filename="material.xacro"/>
-    <xacro:property name="body_length" value="0.22"/>
-    <xacro:property name="body_width" value="0.12"/>
-    <xacro:property name="body_height" value="0.1"/>
-    <xacro:property name="shoulder_length" value="0.043"/>
-    <xacro:property name="shoulder_width" value="0.038"/>
-    <xacro:property name="shoulder_height" value="0.057"/>
-    <xacro:property name="bein_length" value="0.1"/>
-    <xacro:property name="bein_width" value="0.05"/>
-    <xacro:property name="bein_height" value="0.03"/>
-    <xacro:property name="fuss_length" value="0.14"/>
-    <xacro:property name="fuss_width" value="0.045"/>
-    <xacro:property name="fuss_height" value="0.03"/>
-    <xacro:property name="fuss_ballen" value="0.015"/>
-    <xacro:property name="scale" value="0.001 0.001 0.001"/>
-    <link name="base_footprint"/>
-    <link name="base_link">
-        <visual>
-            <origin xyz="-0.013 -0.0325 0.125" rpy="0.0 0.0 ${-pi/2} "/>
-            <geometry>
-               <cylinder radius="${body_height/2}" length="${body_length}"/>
-               <!-- <mesh filename="package://spot_description/meshes/Spot_Chassis.stl" scale="${scale}"/>
-                <box size="${body_length} ${body_width} ${body_height}"/> -->
-            </geometry>
-            <material name="black"/>
-        </visual>
-        <collision>
-            <origin xyz="0.0 0.0 ${body_width/2}" rpy="0.0 ${pi/2} 0.0 "/>
-            <geometry>
-                <cylinder radius="${body_height/2}" length="${body_length}"/>
-                <!--<box size="${body_length} ${body_width} ${body_height}"/> -->
-            </geometry>
-        </collision>
-        <xacro:cylinder_inertia m="0.5" r="${body_height/2}" h="${body_length}"
-                           xyz="0 0 0" rpy="0 0 0"/>
-    </link>
-    <joint name="virtuel_joint" type="fixed">
-        <parent link="base_footprint"/>
-        <child link="base_link"/>
-        <origin xyz="0.0 0.0 0.275" rpy="0.0 0.0 0.0"/>
-    </joint>
-        <!-- Schulter body-->
-    <xacro:macro name="schulter" params="prefix">
-        <link name="${prefix}_schulter_link">
-        <visual>
-            <origin xyz="0.0 0.0 0.0" rpy="0.0 0.0 0.0"/>
-            <geometry>
-                <box size="${shoulder_length} ${shoulder_width} ${shoulder_height}"/>
-            </geometry>
-        </visual>
-        <collision>
-            <origin xyz="0.0 0.0 0.0" rpy="0.0 0.0 0.0"/>
-            <geometry>
-                <box size="${shoulder_length} ${shoulder_width} ${shoulder_height}"/>
-            </geometry>
-        </collision>
-        <xacro:box_inertia m="0.1" l="${shoulder_length}" w="${shoulder_width}" h="${shoulder_height}"
-                           xyz="0 0 0" rpy="0 0 0"/>
-    </link>
-    </xacro:macro>
-    <xacro:schulter prefix="front_r" />
-    <xacro:schulter prefix="front_l" />
-    <xacro:schulter prefix="heck_r" />
-    <xacro:schulter prefix="heck_l" />
-        <!-- Bein body -->
-    <xacro:macro name="bein" params="prefix">
-        <link name="${prefix}_bein_link">
-        <visual>
-            <origin xyz="-0.03 0.0 0.0" rpy="0.0 0.0 0.0"/>
-            <geometry>
-                <box size="${bein_length}  ${bein_width} ${bein_height}"/>
-            </geometry>
-            <material name="white"/>
-        </visual>
-        <collision>
-            <origin xyz="-0.03 0.0 0.0" rpy="0.0 0.0 0.0"/>
-            <geometry>
-                <box size="${bein_length}  ${bein_width} ${bein_height}"/>
-            </geometry>
-        </collision>
-        <xacro:box_inertia m="0.1" l="${bein_length}" w="${bein_width}" h="${bein_height}"
-                           xyz="0 0 0" rpy="0 0 0"/>
-    </link>
-    </xacro:macro>
-    <xacro:bein prefix="front_r" />
-    <xacro:bein prefix="front_l" />
-    <xacro:bein prefix="heck_r" />
-    <xacro:bein prefix="heck_l" />
-        <!-- Fuss body -->
-    <xacro:macro name="fuss" params="prefix">
-        <link name="${prefix}_fuss_link">
-        <visual>
-            <origin xyz="0.055 0.0 0.0" rpy="0.0 0.0 0.0"/>
-            <geometry>
-                <box size="${fuss_length}  ${fuss_width} ${fuss_height}"/>
-            </geometry>
-            <material name="black"/>
-        </visual>
-        <collision>
-            <origin xyz="0.055 0.0 0.0" rpy="0.0 0.0 0.0"/>
-            <geometry>
-                <box size="${fuss_length}  ${fuss_width} ${fuss_height}"/>
-            </geometry>
-        </collision>
-        <xacro:box_inertia m="0.1" l="${fuss_length}" w="${fuss_width}" h="${fuss_height}"
-                           xyz="0 0 0" rpy="0 0 0"/>
-    </link>
-    </xacro:macro>
-    <xacro:fuss prefix="front_r" />
-    <xacro:fuss prefix="front_l" />
-    <xacro:fuss prefix="heck_r" />
-    <xacro:fuss prefix="heck_l" />
-        <!-- Fuss endpoint -->
-    <xacro:macro name="fussb" params="prefix">
-        <link name="${prefix}_fuss_ballen_link">
-        <visual>
-            <origin xyz="-0.015 0.0 0.0" rpy="${pi/2} 0.0 0.0"/>
-            <geometry>
-                <cylinder radius="${fuss_ballen}" length="${fuss_width}"/>
-            </geometry>
-            <material name="black"/>
-        </visual>
-        <collision>
-            <origin xyz="-0.015 0.0 0.0" rpy="${pi/2} 0.0 0.0"/>
-            <geometry>
-                <cylinder radius="${fuss_ballen}" length="${fuss_width}"/>
-            </geometry>
-        </collision>
-        <xacro:cylinder_inertia m="0.01" r="${fuss_ballen}" h="${fuss_width}"
-                           xyz="0 0 0" rpy="0 0 0"/>
-    </link>
-    </xacro:macro>
-    <xacro:fussb prefix="front_r" />
-    <xacro:fussb prefix="front_l" />
-    <xacro:fussb prefix="heck_r" />
-    <xacro:fussb prefix="heck_l" />
-        <!-- Front Rechts-->
-    <joint name="joint_0" type="revolute">
-        <parent link="base_link"/>
-        <child link="front_r_schulter_link"/>
-        <axis xyz="-1 0 0"/>
-        <limit lower="${-pi/4}" upper="${pi/4}" velocity="50.0" effort="1000.0"/>
-        <origin xyz="0.132 -0.0435 ${body_width/2}" rpy="0 0 0"/>
-    </joint>
-    <joint name="joint_1" type="revolute">
-        <parent link="front_r_schulter_link"/>
-        <child link="front_r_bein_link"/>
-        <axis xyz="0 -1 0"/>
-        <limit lower="0" upper="${pi/2}" velocity="50.0" effort="1000.0"/>
-        <origin xyz="0.0 -${shoulder_width/2 + bein_width/2 + 0.003} -0.01" rpy="0 ${-pi/2} 0"/>
-    </joint>
-    <joint name="joint_2" type="revolute">
-        <parent link="front_r_bein_link"/>
-        <child link="front_r_fuss_link"/>
-        <axis xyz="0 1 0"/>
-        <limit lower="0" upper="${pi/2}" velocity="50.0" effort="1000.0"/>
-        <origin xyz="-0.107 0.0 0.03" rpy="0 ${-pi/2} 0"/>
-    </joint>
-    <joint name="rechter_fuss_F_endpoint" type="fixed">
-        <parent link="front_r_fuss_link"/>
-        <child link="front_r_fuss_ballen_link"/>
-        <origin xyz="0.14 0.0 0.0" rpy="0.0 0.0 0.0"/>
-    </joint>
-        <!-- Front Links-->
-    <joint name="joint_3" type="revolute">
-        <parent link="base_link"/>
-        <child link="front_l_schulter_link"/>
-        <axis xyz="1 0 0"/>
-        <limit lower="${-pi/4}" upper="${pi/4}" velocity="50.0" effort="1000.0"/>
-        <origin xyz="0.132 0.0435 ${body_width/2}" rpy="0 0 0"/>
-    </joint>
-    <joint name="joint_4" type="revolute">
-        <parent link="front_l_schulter_link"/>
-        <child link="front_l_bein_link"/>
-        <axis xyz="0 -1 0"/>
-        <limit lower="${-pi/4}" upper="${pi/4}" velocity="50.0" effort="1000.0"/>
-        <origin xyz="0.0 ${shoulder_width/2 + bein_width/2 + 0.003} -0.01" rpy="0 ${-pi/2} 0"/>
-    </joint>
-    <joint name="joint_5" type="revolute">
-        <parent link="front_l_bein_link"/>
-        <child link="front_l_fuss_link"/>
-        <axis xyz="0 1 0"/>
-        <limit lower="${-pi/4}" upper="${pi/4}" velocity="50.0" effort="1000.0"/>
-        <origin xyz="-0.107 0.0 0.03" rpy="0 ${-pi/2} 0"/>
-    </joint>
-    <joint name="linker_fuss_F_endpoint" type="fixed">
-        <parent link="front_l_fuss_link"/>
-        <child link="front_l_fuss_ballen_link"/>
-        <origin xyz="0.14 0.0 0.0" rpy="0.0 0.0 0.0"/>
-    </joint>
-        <!-- Heck Rechts-->
-    <joint name="joint_6" type="revolute">
-        <parent link="base_link"/>
-        <child link="heck_r_schulter_link"/>
-        <axis xyz="-1 0 0"/>
-        <limit lower="${-pi/4}" upper="${pi/4}" velocity="50.0" effort="1000.0"/>
-        <origin xyz="-0.134 -0.0435 ${body_width/2}" rpy="0 0 0"/>
-    </joint>
-    <joint name="joint_7" type="revolute">
-        <parent link="heck_r_schulter_link"/>
-        <child link="heck_r_bein_link"/>
-        <axis xyz="0 -1 0"/>
-        <limit lower="${-pi/4}" upper="${pi/4}" velocity="50.0" effort="1000.0"/>
-        <origin xyz="0.0 -${shoulder_width/2 + bein_width/2 + 0.003} -0.01" rpy="0 ${-pi/2} 0"/>
-    </joint>
-    <joint name="joint_8" type="revolute">
-        <parent link="heck_r_bein_link"/>
-        <child link="heck_r_fuss_link"/>
-        <axis xyz="0 1 0"/>
-        <limit lower="${-pi/4}" upper="${pi/4}" velocity="50.0" effort="1000.0"/>
-        <origin xyz="-0.107 0.0 0.03" rpy="0 ${-pi/2} 0"/>
-    </joint>
-    <joint name="rechter_fuss_H_endpoint" type="fixed">
-        <parent link="heck_r_fuss_link"/>
-        <child link="heck_r_fuss_ballen_link"/>
-        <origin xyz="0.14 0.0 0.0" rpy="0.0 0.0 0.0"/>
-    </joint>
-        <!-- Heck Links-->
-    <joint name="joint_9" type="revolute">
-        <parent link="base_link"/>
-        <child link="heck_l_schulter_link"/>
-        <axis xyz="1 0 0"/>
-        <limit lower="${-pi/4}" upper="${pi/4}" velocity="50.0" effort="1000.0"/>
-        <origin xyz="-0.134 0.0435 ${body_width/2}" rpy="0 0 0"/>
-    </joint>
-    <joint name="joint_10" type="revolute">
-        <parent link="heck_l_schulter_link"/>
-        <child link="heck_l_bein_link"/>
-        <axis xyz="0 -1 0"/>
-        <limit lower="${-pi/4}" upper="${pi/4}" velocity="50.0" effort="1000.0"/>
-        <origin xyz="0.0 ${shoulder_width/2 + bein_width/2 + 0.003} -0.01" rpy="0 ${-pi/2} 0"/>
-    </joint>
-    <joint name="joint_11" type="revolute">
-        <parent link="heck_l_bein_link"/>
-        <child link="heck_l_fuss_link"/>
-        <axis xyz="0 1 0"/>
-        <limit lower="${-pi/4}" upper="${pi/4}" velocity="50.0" effort="1000.0"/>
-        <origin xyz="-0.107 0.0 0.03" rpy="0 ${-pi/2} 0"/>
-    </joint>
-    <joint name="linker_fuss_H_endpoint" type="fixed">
-        <parent link="heck_l_fuss_link"/>
-        <child link="heck_l_fuss_ballen_link"/>
-        <origin xyz="0.14 0.0 0.0" rpy="0.0 0.0 0.0"/>
-    </joint>
+    <xacro:include filename="spot_core.xacro"/>
+    <xacro:include filename="gazebo.xacro"/>
+    <xacro:include filename="ros2_control.xacro"/>
 </robot>
