Commit message: ros2 control in work

File: spot_description/urdf/gazebo.xacro (robot description, xacro)
@@ -5,5 +5,5 @@
             <robot_param>robot_description</robot_param>
             <robot_param_node>robot_state_publisher</robot_param_node>
-            <parameters></parameters>
+            <parameters>$(find spot_controller)/config/spot_controllers.yaml</parameters>
         </plugin>
     </gazebo>

File: spot_description/urdf/ros2_control.xacro (robot description, xacro)
@@ -4,10 +4,10 @@
     <ros2_control name="RobotSystem" type="system">
         <hardware>
-            <plugin> gazebo_ros2_control/GazeboSystem </plugin>
+            <plugin>gazebo_ros2_control/GazeboSystem</plugin>
         </hardware>
         <joint name="joint_0">
             <command_interface name="position">
-                <param name="min">${-PI/2}</param>
-                <param name="max">${PI/2}</param>
+                <param name="min">${-PI/4}</param>
+                <param name="max">${PI/4}</param>
             </command_interface>
             <state_interface name="position" />
@@ -15,6 +15,6 @@
         <joint name="joint_1">
             <command_interface name="position">
-                <param name="min">${-PI/2}</param>
-                <param name="max">${PI/2}</param>
+                <param name="min">${-PI/4}</param>
+                <param name="max">${PI/4}</param>
             </command_interface>
             <state_interface name="position" />
@@ -22,6 +22,6 @@
         <joint name="joint_2">
             <command_interface name="position">
-                <param name="min">${-PI/2}</param>
-                <param name="max">${PI/2}</param>
+                <param name="min">${-PI/4}</param>
+                <param name="max">${PI/4}</param>
             </command_interface>
             <state_interface name="position" />
@@ -29,6 +29,6 @@
         <joint name="joint_3">
             <command_interface name="position">
-                <param name="min">${-PI/2}</param>
-                <param name="max">${PI/2}</param>
+                <param name="min">${-PI/4}</param>
+                <param name="max">${PI/4}</param>
             </command_interface>
             <state_interface name="position" />
@@ -36,6 +36,6 @@
         <joint name="joint_4">
             <command_interface name="position">
-                <param name="min">${-PI/2}</param>
-                <param name="max">${PI/2}</param>
+                <param name="min">${-PI/4}</param>
+                <param name="max">${PI/4}</param>
             </command_interface>
             <state_interface name="position" />
@@ -43,6 +43,6 @@
         <joint name="joint_5">
             <command_interface name="position">
-                <param name="min">${-PI/2}</param>
-                <param name="max">${PI/2}</param>
+                <param name="min">${-PI/4}</param>
+                <param name="max">${PI/4}</param>
             </command_interface>
             <state_interface name="position" />
@@ -50,6 +50,6 @@
         <joint name="joint_6">
             <command_interface name="position">
-                <param name="min">${-PI/2}</param>
-                <param name="max">${PI/2}</param>
+                <param name="min">${-PI/4}</param>
+                <param name="max">${PI/4}</param>
             </command_interface>
             <state_interface name="position" />
@@ -57,6 +57,6 @@
         <joint name="joint_7">
             <command_interface name="position">
-                <param name="min">${-PI/2}</param>
-                <param name="max">${PI/2}</param>
+                <param name="min">${-PI/4}</param>
+                <param name="max">${PI/4}</param>
             </command_interface>
             <state_interface name="position" />
@@ -64,6 +64,6 @@
         <joint name="joint_8">
             <command_interface name="position">
-                <param name="min">${-PI/2}</param>
-                <param name="max">${PI/2}</param>
+                <param name="min">${-PI/4}</param>
+                <param name="max">${PI/4}</param>
             </command_interface>
             <state_interface name="position" />
@@ -71,6 +71,6 @@
         <joint name="joint_9">
             <command_interface name="position">
-                <param name="min">${-PI/2}</param>
-                <param name="max">${PI/2}</param>
+                <param name="min">${-PI/4}</param>
+                <param name="max">${PI/4}</param>
             </command_interface>
             <state_interface name="position" />
@@ -78,6 +78,6 @@
         <joint name="joint_10">
             <command_interface name="position">
-                <param name="min">${-PI/2}</param>
-                <param name="max">${PI/2}</param>
+                <param name="min">${-PI/4}</param>
+                <param name="max">${PI/4}</param>
             </command_interface>
             <state_interface name="position" />
@@ -85,6 +85,6 @@
         <joint name="joint_11">
             <command_interface name="position">
-                <param name="min">${-PI/2}</param>
-                <param name="max">${PI/2}</param>
+                <param name="min">${-PI/4}</param>
+                <param name="max">${PI/4}</param>
             </command_interface>
             <state_interface name="position" />

File: spot_description/urdf/spot_core.xacro (robot description, xacro)
@@ -159,5 +159,5 @@
         <child link="front_r_bein_link"/>
         <axis xyz="0 -1 0"/>
-        <limit lower="0" upper="${pi/2}" velocity="50.0" effort="1000.0"/>
+        <limit lower="${-pi/4}" upper="${pi/4}" velocity="50.0" effort="1000.0"/>
         <origin xyz="0.0 -${shoulder_width/2 + bein_width/2 + 0.003} -0.01" rpy="0 ${-pi/2} 0"/>
     </joint>
@@ -166,5 +166,5 @@
         <child link="front_r_fuss_link"/>
         <axis xyz="0 1 0"/>
-        <limit lower="0" upper="${pi/2}" velocity="50.0" effort="1000.0"/>
+        <limit lower="${-pi/4}" upper="${pi/4}" velocity="50.0" effort="1000.0"/>
         <origin xyz="-0.107 0.0 0.03" rpy="0 ${-pi/2} 0"/>
     </joint>
